File: pcb/phalanx.kicad_pcb (KiCad board)
At the start: 2 copper layers, 187.2 x 77.2 mm, 113 parts, among them J1 TYPE-C-31-M-12, J2 PJ-320A, J3 PJ-320A, K0_0 SW_KEY, K0_1 SW_KEY, K0_2 SW_KEY, K0_3 SW_KEY, K0_4 SW_KEY, K0_5 SW_KEY, K0_6 SW_KEY, K0_7 SW_KEY, K1_0 SW_KEY, K1_1 SW_KEY, K1_2 SW_KEY, K1_3 SW_KEY, K1_4 SW_KEY, K1_5 SW_KEY, K1_6 SW_KEY, K1_7 SW_KEY, K2_0 SW_KEY, K2_1 SW_KEY, K2_2 SW_KEY, K2_3 SW_KEY, K2_4 SW_KEY, K2_5 SW_KEY, K2_6 SW_KEY, K2_7 SW_KEY, K3_2 SW_KEY, K3_3 SW_KEY, K3_4 SW_KEY, K3_5 SW_KEY, Q1 PDTC123JT,215, SW2 B3U-1000P, U1 STM32F072CBT6, U2 MCP23017-E/SO, U3 SRV05-4, U4 MCP1700T-3302E/TT

Commit message: 🚨 Fix DRC (design rule check) warnings
Routing:
- net GND1: track 0.59 -> 6.41 mm, vias 0 -> 4
Changed lines of the file:
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@@
     (fp_line (start 1 0.625) (end -1 0.625)
       (stroke (width 0.1) (type solid)) (layer "F.Fab"))
-    (pad "1" smd roundrect (at -0.9125 0 90) (size 1.025 1.4) (layers "F.Cu" "F.Paste" "F.Mask") (roundrect_rratio 0.243902439)
+    (pad "1" smd roundrect (at -0.9125 0 90) (size 1.025 1.4) (layers "F.Cu" "F.Paste" "F.Mask") (roundrect_rratio 0.243902)
       (net 45 "Net-(J1-CC1)") (pintype "passive"))
-    (pad "2" smd roundrect (at 0.9125 0 90) (size 1.025 1.4) (layers "F.Cu" "F.Paste" "F.Mask") (roundrect_rratio 0.243902439)
+    (pad "2" smd roundrect (at 0.9125 0 90) (size 1.025 1.4) (layers "F.Cu" "F.Paste" "F.Mask") (roundrect_rratio 0.243902)
       (net 1 "GND") (pintype "passive"))
     (model "${KICAD6_3DMODEL_DIR}/Resistor_SMD.3dshapes/R_0805_2012Metric.wrl"
@@
     (fp_line (start 1 0.625) (end -1 0.625)
       (stroke (width 0.1) (type solid)) (layer "F.Fab"))
-    (pad "1" smd roundrect (at -0.9125 0 90) (size 1.025 1.4) (layers "F.Cu" "F.Paste" "F.Mask") (roundrect_rratio 0.243902439)
+    (pad "1" smd roundrect (at -0.9125 0 90) (size 1.025 1.4) (layers "F.Cu" "F.Paste" "F.Mask") (roundrect_rratio 0.243902)
       (net 3 "VDD") (pintype "passive"))
-    (pad "2" smd roundrect (at 0.9125 0 90) (size 1.025 1.4) (layers "F.Cu" "F.Paste" "F.Mask") (roundrect_rratio 0.243902439)
+    (pad "2" smd roundrect (at 0.9125 0 90) (size 1.025 1.4) (layers "F.Cu" "F.Paste" "F.Mask") (roundrect_rratio 0.243902)
       (net 64 "Net-(U2-~{RESET})") (pintype "passive"))
     (model "${KICAD6_3DMODEL_DIR}/Resistor_SMD.3dshapes/R_0805_2012Metric.wrl"
@@
     (fp_line (start 1 0.625) (end -1 0.625)
       (stroke (width 0.1) (type solid)) (layer "F.Fab"))
-    (pad "1" smd roundrect (at -0.9125 0 270) (size 1.025 1.4) (layers "F.Cu" "F.Paste" "F.Mask") (roundrect_rratio 0.243902439)
+    (pad "1" smd roundrect (at -0.9125 0 270) (size 1.025 1.4) (layers "F.Cu" "F.Paste" "F.Mask") (roundrect_rratio 0.243902)
       (net 6 "BOOT0") (pintype "passive"))
-    (pad "2" smd roundrect (at 0.9125 0 270) (size 1.025 1.4) (layers "F.Cu" "F.Paste" "F.Mask") (roundrect_rratio 0.243902439)
+    (pad "2" smd roundrect (at 0.9125 0 270) (size 1.025 1.4) (layers "F.Cu" "F.Paste" "F.Mask") (roundrect_rratio 0.243902)
       (net 1 "GND") (pintype "passive"))
     (model "${KICAD6_3DMODEL_DIR}/Resistor_SMD.3dshapes/R_0805_2012Metric.wrl"
@@
     (fp_line (start 1 0.625) (end -1 0.625)
       (stroke (width 0.1) (type solid)) (layer "F.Fab"))
-    (pad "1" smd roundrect (at -0.9125 0 90) (size 1.025 1.4) (layers "F.Cu" "F.Paste" "F.Mask") (roundrect_rratio 0.243902439)
+    (pad "1" smd roundrect (at -0.9125 0 90) (size 1.025 1.4) (layers "F.Cu" "F.Paste" "F.Mask") (roundrect_rratio 0.243902)
       (net 55 "i2c_scl_right") (pintype "passive"))
-    (pad "2" smd roundrect (at 0.9125 0 90) (size 1.025 1.4) (layers "F.Cu" "F.Paste" "F.Mask") (roundrect_rratio 0.243902439)
+    (pad "2" smd roundrect (at 0.9125 0 90) (size 1.025 1.4) (layers "F.Cu" "F.Paste" "F.Mask") (roundrect_rratio 0.243902)
       (net 3 "VDD") (pintype "passive"))
     (model "${KICAD6_3DMODEL_DIR}/Resistor_SMD.3dshapes/R_0805_2012Metric.wrl"
@@
     (fp_line (start 1 0.625) (end -1 0.625)
       (stroke (width 0.1) (type solid)) (layer "F.Fab"))
-    (pad "1" smd roundrect (at -0.9125 0 270) (size 1.025 1.4) (layers "F.Cu" "F.Paste" "F.Mask") (roundrect_rratio 0.243902439)
+    (pad "1" smd roundrect (at -0.9125 0 270) (size 1.025 1.4) (layers "F.Cu" "F.Paste" "F.Mask") (roundrect_rratio 0.243902)
       (net 4 "+5V") (pintype "passive"))
-    (pad "2" smd roundrect (at 0.9125 0 270) (size 1.025 1.4) (layers "F.Cu" "F.Paste" "F.Mask") (roundrect_rratio 0.243902439)
+    (pad "2" smd roundrect (at 0.9125 0 270) (size 1.025 1.4) (layers "F.Cu" "F.Paste" "F.Mask") (roundrect_rratio 0.243902)
       (net 1 "GND") (pintype "passive"))
     (model "${KICAD6_3DMODEL_DIR}/Resistor_SMD.3dshapes/R_0805_2012Metric.wrl"
@@
     (fp_line (start 1 0.625) (end -1 0.625)
       (stroke (width 0.1) (type solid)) (layer "F.Fab"))
-    (pad "1" smd roundrect (at -0.9125 0 90) (size 1.025 1.4) (layers "F.Cu" "F.Paste" "F.Mask") (roundrect_rratio 0.243902439)
+    (pad "1" smd roundrect (at -0.9125 0 90) (size 1.025 1.4) (layers "F.Cu" "F.Paste" "F.Mask") (roundrect_rratio 0.243902)
       (net 1 "GND") (pintype "passive"))
-    (pad "2" smd roundrect (at 0.9125 0 90) (size 1.025 1.4) (layers "F.Cu" "F.Paste" "F.Mask") (roundrect_rratio 0.243902439)
+    (pad "2" smd roundrect (at 0.9125 0 90) (size 1.025 1.4) (layers "F.Cu" "F.Paste" "F.Mask") (roundrect_rratio 0.243902)
       (net 49 "Net-(J1-CC2)") (pintype "passive"))
     (model "${KICAD6_3DMODEL_DIR}/Resistor_SMD.3dshapes/R_0805_2012Metric.wrl"
@@
     (fp_line (start 1 0.625) (end -1 0.625)
       (stroke (width 0.1) (type solid)) (layer "F.Fab"))
-    (pad "1" smd roundrect (at -0.9125 0 270) (size 1.025 1.4) (layers "F.Cu" "F.Paste" "F.Mask") (roundrect_rratio 0.243902439)
+    (pad "1" smd roundrect (at -0.9125 0 270) (size 1.025 1.4) (layers "F.Cu" "F.Paste" "F.Mask") (roundrect_rratio 0.243902)
       (net 2 "+3.3V") (pintype "passive"))
-    (pad "2" smd roundrect (at 0.9125 0 270) (size 1.025 1.4) (layers "F.Cu" "F.Paste" "F.Mask") (roundrect_rratio 0.243902439)
+    (pad "2" smd roundrect (at 0.9125 0 270) (size 1.025 1.4) (layers "F.Cu" "F.Paste" "F.Mask") (roundrect_rratio 0.243902)
       (net 1 "GND") (pintype "passive"))
     (model "${KICAD6_3DMODEL_DIR}/Resistor_SMD.3dshapes/R_0805_2012Metric.wrl"
@@
     (fp_line (start 1 0.625) (end -1 0.625)
       (stroke (width 0.1) (type solid)) (layer "F.Fab"))
-    (pad "1" smd roundrect (at -0.9125 0 90) (size 1.025 1.4) (layers "F.Cu" "F.Paste" "F.Mask") (roundrect_rratio 0.243902439)
+    (pad "1" smd roundrect (at -0.9125 0 90) (size 1.025 1.4) (layers "F.Cu" "F.Paste" "F.Mask") (roundrect_rratio 0.243902)
       (net 54 "i2c_sda_right") (pintype "passive"))
-    (pad "2" smd roundrect (at 0.9125 0 90) (size 1.025 1.4) (layers "F.Cu" "F.Paste" "F.Mask") (roundrect_rratio 0.243902439)
+    (pad "2" smd roundrect (at 0.9125 0 90) (size 1.025 1.4) (layers "F.Cu" "F.Paste" "F.Mask") (roundrect_rratio 0.243902)
       (net 3 "VDD") (pintype "passive"))
     (model "${KICAD6_3DMODEL_DIR}/Resistor_SMD.3dshapes/R_0805_2012Metric.wrl"
@@
   (segment (start 65.8725 92.395) (end 65.855 92.4125) (width 0.5) (layer "F.Cu") (net 102))
   (segment (start 71.68 101.05) (end 71.53 101.2) (width 0.5) (layer "F.Cu") (net 102))
+  (segment (start 73.025 87.66) (end 71.08 87.66) (width 0.3) (layer "F.Cu") (net 102))
+  (segment (start 73.025 88.93) (end 71.09 88.93) (width 0.3) (layer "F.Cu") (net 102))
   (segment (start 71.53 101.2) (end 71.28 101.45) (width 0.3) (layer "F.Cu") (net 102))
+  (segment (start 73.025 90.2) (end 71.09 90.2) (width 0.3) (layer "F.Cu") (net 102))
+  (via (at 71.09 88.93) (size 0.8) (drill 0.4) (layers "F.Cu" "B.Cu") (net 102))
+  (via (at 71.09 90.2) (size 0.8) (drill 0.4) (layers "F.Cu" "B.Cu") (net 102))
+  (via (at 71.08 87.66) (size 0.8) (drill 0.4) (layers "F.Cu" "B.Cu") (net 102))
+  (via (at 68.88 101.43) (size 0.8) (drill 0.4) (layers "F.Cu" "B.Cu") (net 102))
   (zone (net 44) (net_name "VCC") (layer "F.Cu") (hatch edge 0.508)
     (priority 6)

Commit message: ✨ Add updated PCB files
Parts:
- removed the C8 at (65.9, 93.3)
- removed the C9 at (63.4, 93.3)
- removed the G*** at (68.4, 63.8)
- removed the R1 at (73.4, 93.3)
- removed R7, R8: 4k7, Resistor_SMD:R_0805_2012Metric
- removed the U2 at (68.4, 81.9)
- added D4: LED, LED_SMD:LED_0603_1608Metric, F.Cu at (223.0, 73.7)
- added R5: 51, Resistor_SMD:R_0805_2012Metric, F.Cu at (225.9, 74.6)
- C1: renamed from C10; value 1uF -> 1u
- C10: renamed from C7; value 10u -> 10n
- C2: renamed from C11; value 1uF -> 1u
- J2, J3: value PJ-320A -> 8P8C; footprint library:TRRS-PJ-320A -> library:RJ45
- moved R1 75.8 mm to (159.9, 65.5), turned to 0 degrees
- moved R2 74.4 mm to (152.6, 65.5), turned to 0 degrees
- moved G*** 74.0 mm to (139.9, 60.3)
- moved J1 72.9 mm to (156.2, 58.8)
- moved D1 66.8 mm to (164.6, 57.6)
- moved U2 65.5 mm to (164.9, 64.8)
- moved F1 57.8 mm to (164.7, 60.9), turned to 0 degrees
- moved J3 37.5 mm to (71.6, 63.5), turned to 180 degrees
- moved J2 36.0 mm to (232.7, 63.5), turned to 180 degrees
- moved C7 30.0 mm to (222.9, 95.5), turned to 180 degrees
- moved R3 27.6 mm to (235.1, 68.5), turned to 0 degrees
- moved C1 24.3 mm to (235.1, 71.0), turned to 0 degrees
- moved D3 21.8 mm to (228.7, 103.6)
- moved R6 20.9 mm to (222.2, 104.2)
- moved U1 19.8 mm to (235.1, 74.4), turned to 90 degrees
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- renumbered C5 to C11, C13 to C3, C12 to C4, C1 to C5, C4 to C6, C3 to C7, C2 to C8, C6 to C9, D0_4 to D4_0, D0_5 to D4_1, D0_6 to D4_2, D0_7 to D4_3, D1_4 to D5_0, D1_5 to D5_1, D1_6 to D5_2, D1_7 to D5_3, D2_4 to D6_0, D2_5 to D6_1, D2_6 to D6_2, D2_7 to D6_3, D3_4 to D7_0, D3_5 to D7_1, K0_4 to K4_0, K0_5 to K4_1, K0_6 to K4_2, K0_7 to K4_3, K1_4 to K5_0, K1_5 to K5_1, K1_6 to K5_2, K1_7 to K5_3, K2_4 to K6_0, K2_5 to K6_1, K2_6 to K6_2, K2_7 to K6_3, K3_4 to K7_0, K3_5 to K7_1, R2 to R1, R3 to R2, R4 to R3, R5 to R4, SW2 to SW1, U4 to U1, U3 to U2, U1 to U3
Connections:
- net /row0_0 renamed /row0
- C5 pad 1: GND -> +3.3V
- C5 pad 2: +3.3V -> GND
- C6 pad 1: +3.3V -> GND
- C6 pad 2: GND -> +3.3V
- C7 pad 1: GND -> +3.3V
- C7 pad 2: +3.3V -> GND
- C8 pad 1: +3.3V -> GND
- C8 pad 2: GND -> +3.3V
- C9 pad 1: +3.3V -> GND
- C9 pad 2: GND -> +3.3V
- D1_0 pad 1: /row0_1 -> /row1
- D1_1 pad 1: /row0_1 -> /row1
- D1_2 pad 1: /row0_1 -> /row1
- D1_3 pad 1: /row0_1 -> /row1
- D2_0 pad 1: /row0_2 -> /row2
- D2_1 pad 1: /row0_2 -> /row2
- D2_2 pad 1: /row0_2 -> /row2
- D2_3 pad 1: /row0_2 -> /row2
- D3_2 pad 1: /row0_3 -> /row3
- D3_3 pad 1: /row0_3 -> /row3
- D4_0 pad 1: /row1_0 -> /row4R
- D4_1 pad 1: /row1_0 -> /row4R
- D4_2 pad 1: /row1_0 -> /row4R
- D4_3 pad 1: /row1_0 -> /row4R
- D5_0 pad 1: /row1_1 -> /row5R
- D5_1 pad 1: /row1_1 -> /row5R
- D5_2 pad 1: /row1_1 -> /row5R
- D5_3 pad 1: /row1_1 -> /row5R
- D6_0 pad 1: /row1_2 -> /row6R
- D6_1 pad 1: /row1_2 -> /row6R
- D6_2 pad 1: /row1_2 -> /row6R
- D6_3 pad 1: /row1_2 -> /row6R
- D7_0 pad 1: /row1_3 -> /row7R
- D7_1 pad 1: /row1_3 -> /row7R
- K4_0 pad 1: /col4 -> /col0R
- K4_1 pad 1: /col5 -> /col1R
- K4_2 pad 1: /col6 -> /col2R
- K4_3 pad 1: /col7 -> /col3R
- K5_0 pad 1: /col4 -> /col0R
- K5_1 pad 1: /col5 -> /col1R
- K5_2 pad 1: /col6 -> /col2R
- K5_3 pad 1: /col7 -> /col3R
- K6_0 pad 1: /col4 -> /col0R
- K6_1 pad 1: /col5 -> /col1R
- K6_2 pad 1: /col6 -> /col2R
- K6_3 pad 1: /col7 -> /col3R
- K7_0 pad 1: /col4 -> /col0R
- K7_1 pad 1: /col5 -> /col1R
- U3 pad 12: /row0_3 -> unconnected-(U3-PA2-Pad12)
- U3 pad 21: i2c_scl -> unconnected-(U3-PB10-Pad21)
- U3 pad 22: i2c_sda -> /col1
- U3 pad 25: unconnected-(U1-PB12-Pad25) -> /col2
- U3 pad 26: unconnected-(U1-PB13-Pad26) -> /col3
- U3 pad 27: unconnected-(U1-PB14-Pad27) -> /row5
- U3 pad 28: unconnected-(U1-PB15-Pad28) -> /row6
- U3 pad 29: unconnected-(U1-PA8-Pad29) -> /row7
- U3 pad 30: unconnected-(U1-PA9-Pad30) -> /col0
- U3 pad 31: unconnected-(U1-PA10-Pad31) -> /row4
- U3 pad 38: /col3 -> /row1
- U3 pad 39: /col2 -> /row2
- U3 pad 40: /col1 -> /row3
- U3 pad 41: /col0 -> unconnected-(U3-PB5-Pad41)
- U3 pad 42: /row0_1 -> unconnected-(U3-PB6-Pad42)
- U3 pad 43: /row0_2 -> unconnected-(U3-PB7-Pad43)
Routing:
- net /col3R: track 0.00 -> 117.2 mm
- net /col1R: track 0.00 -> 116.4 mm
- net /col7: track 114.9 -> 0.00 mm
- net /col5: track 114.6 -> 0.00 mm
- net /row6R: track 0.00 -> 101.8 mm
- net /row1_0: track 95.3 -> 0.00 mm
- net /row0_2: track 94.3 -> 0.00 mm
- net /row4R: track 0.00 -> 94.1 mm
- net /col6: track 93.2 -> 0.00 mm
- net /col2R: track 0.00 -> 91.8 mm
- net /col0R: track 0.00 -> 88.0 mm
- net /USB_D-: track 19.6 -> 107.2 mm, vias 2 -> 4
- net /row5R: track 0.00 -> 87.0 mm
- net /row1_2: track 86.1 -> 0.00 mm
- net /row1: track 0.00 -> 84.7 mm
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- added copper zone on B.Cu, net (none)
- added copper zone on F.Cu, net (none)
- removed copper zone on B.Cu, net GND1
- removed copper zone on F.Cu, net GND1
- removed copper zone on F.Cu, net VCC
Other:
- outline, holes or cut-outs redrawn
- board text added: "v0.1.0"

Commit message: 🐛 Increase resistance on pwr LED
Parts:
- R5: value 51 -> 1k
Changed lines of the file:
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@@
     (descr "Resistor SMD 0805 (2012 Metric), square (rectangular) end terminal, IPC_7351 nominal, (Body size source: IPC-SM-782 page 72, https://www.pcb-3d.com/wordpress/wp-content/uploads/ipc-sm-782a_amendment_1_and_2.pdf), generated with kicad-footprint-generator")
     (tags "resistor")
-    (property "LCSC Part" " C25318")
+    (property "LCSC Part" "C17513")
     (property "Part Name" "Resistor")
     (property "Sheetfile" "phalanx.kicad_sch")
@@
         (effects (font (size 1 1) (thickness 0.15)))
     )
-    (fp_text value "51" (at 0 1.65 90) (layer "F.Fab")
+    (fp_text value "1k" (at 0 1.65 90) (layer "F.Fab")
         (effects (font (size 1 1) (thickness 0.15)))
     )

Commit message: 💚 Fix CI/build
Update files from KiCad 7 to KiCad 8 and fix all DRC/ERC errors.
Routing:
- net unconnected-(J1-SHIELD-PadS1)_0: track 17.0 -> 0.00 mm
